File: headphones/headphones.kicad_pcb (KiCad board)
At the start: 4 copper layers, 191 parts, among them J1 UJ20-C-H-G-SMT-1-P16-TR, J2 Conn_ARM_SWD_TagConnect_TC203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, P1 S2B-PH-SM4-TB, SW1 OS102011MS2QN1, SW2 OS102011MS2QN1, SW3 SW_MEC_5E, SW4 SW_MEC_5E, SW5 OS102011MS2QN1, SW6 OS102011MS2QN1, U1 BQ24133RGY, U10 TLV9062IDR, U2 AP2127N-3.0, U3 STM32WB55CCUx, U4 TLV9064IDR, U5 TLV9062IDR, U6 TLV9062IDR, U7 TLV9064IDR, U8 NAU8402WG, U9 TLV9061IDBVR, X1 NX2016SA-32MHZ-EXS00A-CS06654

Commit message: Final Rev2 before purchase
Parts:
- removed C29, C30, C31, C32, C33, C34, C40, C41, C42, C43, C44, C45, C46, C47, C48, C53, C54, C55, C56: 10uF, Capacitor_SMD:C_0603_1608Metric
- removed C39, C49, C50, C51: 330uF, Capacitor_SMD:C_1210_3225Metric
- removed C52: 2.2uF, Capacitor_SMD:C_0603_1608Metric
- removed C57: 220nF, Capacitor_SMD:C_0402_1005Metric
- removed C58, C59: 4.7uF, Capacitor_SMD:C_0402_1005Metric
- removed R26, R34, R55, R59: 390, Resistor_SMD:R_0402_1005Metric
- removed R27, R35, R56, R60: 91k, Resistor_SMD:R_0603_1608Metric
- removed R28, R36, R57, R61: 6.2k, Resistor_SMD:R_0603_1608Metric
- removed R29, R30, R31, R46: PTN16-A01220K1B2, Pot2gang_PTN16_A01220K1B2:POT_PTN16-A01220K1B2
- removed R32, R47, R48, R66, R67: 20k, Resistor_SMD:R_0402_1005Metric
- removed R33, R54, R58: 2.4k, Resistor_SMD:R_0402_1005Metric
- removed R37, R38, R39, R49, R50, R51: 1.3k, Resistor_SMD:R_0402_1005Metric
- removed R40, R42, R44, R52, R62, R64, R68, R69, R70, R71, R72, R73, R74, R75: 10k, Resistor_SMD:R_0402_1005Metric
- removed R41, R43, R45, R53, R63, R65: 1k, Resistor_SMD:R_0402_1005Metric
- removed SW5, SW6: OS102011MS2QN1, SPDT_OS102011MS2QN1:SPDT_OS102011_CNK
- removed TP1, TP12, TP13, TP14, TP15, TP16, TP17, TP2, TP22, TP23, TP4, TP5, TP6, TP7: TestPoint, TestPoint:TestPoint_Pad_D1.5mm
- removed TP18: +LDriver, TestPoint:TestPoint_Pad_D1.5mm
- removed TP19: -LDriver, TestPoint:TestPoint_Pad_D1.5mm
- removed TP20: +RDriver, TestPoint:TestPoint_Pad_D1.5mm
- removed TP21: -RDriver, TestPoint:TestPoint_Pad_D1.5mm
- removed U10, U5, U6: TLV9062IDR, 2OpAmp_TLV9062IDR:D0008A_M
- removed U7: TLV9064IDR, 4OpAmp_TLV9064IDR:D0014A_N
- removed U8: NAU8402WG, DAC_NAU8402WG:TSSOP16_NAU8402_NUV
- removed U9: TLV9061IDBVR, 1OpAmp_TLV9061IDBVR:DBV5_TEX
- added 3.0V: TestPoint, TestPoint:TestPoint_Pad_D1.5mm, F.Cu at (126.0, 116.5)
- added Batt: TestPoint, TestPoint:TestPoint_Pad_D1.5mm, F.Cu at (179.8, 116.1)
- added S1: SLW-1478144-5A-S-D, SP4T_SLW_1478144_5A_S_D:SW_SLW-1478144-5A-S-D, F.Cu at (170.6, 76.9)
- added VDDA: TestPoint, TestPoint:TestPoint_Pad_D1.5mm, F.Cu at (131.8, 92.6)
- added gnd: , , F.Cu at (118.6, 120.7)
- C1, C12, C18, C19, C2, C20, C21, C22, C3, C5, C7, C8: footprint Capacitor_SMD:C_0402_1005Metric -> Capacitor_SMD:C_0603_1608Metric
- C10: value 1uF -> 0.1uF
- C11: value 0.1uF -> 1uF; footprint Capacitor_SMD:C_0402_1005Metric -> Capacitor_SMD:C_0603_1608Metric
- C16: value 10u -> 2.2uF
- C17: value 0.1u -> 10u; footprint Capacitor_SMD:C_0402_1005Metric -> Capacitor_SMD:C_0603_1608Metric
- C23: value 10n -> 0.1u; footprint Capacitor_SMD:C_0402_1005Metric -> Capacitor_SMD:C_0603_1608Metric
- C24: value 1u -> 220nF; footprint Capacitor_SMD:C_0402_1005Metric -> Capacitor_SMD:C_0603_1608Metric
- C25: value 1u -> 4.7uF; footprint Capacitor_SMD:C_0402_1005Metric -> Capacitor_SMD:C_0603_1608Metric
- C26: value 10uF -> 4.7uF
- C27: value 10uF -> 10n
- C28, C35: value 10uF -> 1u
- C36: value 10uF -> 0.1u
- C37: value 330uF -> 1uF; footprint Capacitor_SMD:C_1210_3225Metric -> Capacitor_SMD:C_0603_1608Metric
- C38: value 330uF -> 2.7pF; footprint Capacitor_SMD:C_1210_3225Metric -> Capacitor_SMD:C_0402_1005Metric
- J1: footprint UJ20-C-H-G-SMT-1-P16-TR:SAMESKY_UJ20-C-H-G-SMT-1-P16-TR -> USBC_Connector:SAMESKY_UJ20-C-H-G-SMT-1-P16-TR
- R1, R11, R12, R13, R14, R15, R16, R17, R18, R19, R2, R20, R22, R23, R3, R4, R6, R7, R8, TH1: footprint Resistor_SMD:R_0402_1005Metric -> Resistor_SMD:R_0603_1608Metric
- R24: value 20k -> P120PK-Y25BR10K; footprint Resistor_SMD:R_0402_1005Metric -> Pot1gang10k_P120PK_Y25BR10K:POT_P120PK-x25_TTE
- R25: value 2.4k -> 0
- TP10: value TestPoint -> +RDriver
- TP11: value TestPoint -> -RDriver
- TP8: value TestPoint -> +LDriver
- TP9: value TestPoint -> -LDriver
- U3: value STM32WB55CCUx -> NAU8402WG; footprint Package_DFN_QFN:QFN-48-1EP_7x7mm_P0.5mm_EP5.6x5.6mm -> DAC_NAU8402WG:TSSOP16_NAU8402_NUV
- U4: value TLV9064IDR -> STM32WB55CCUx; footprint 4OpAmp_TLV9064IDR:D0014A_N -> Package_DFN_QFN:QFN-48-1EP_7x7mm_P0.5mm_EP5.6x5.6mm
- moved C37 162.4 mm to (167.5, 117.3), turned to -90 degrees
- moved J1 161.7 mm to (182.3, 99.7), turned to 90 degrees
- moved SW1 146.5 mm to (175.8, 117.8), turned to -90 degrees
- moved R6 136.7 mm to (178.6, 92.1), turned to 90 degrees
- moved C10 133.3 mm to (154.0, 95.6), turned to -90 degrees
- moved C13 132.3 mm to (154.0, 113.8), turned to 180 degrees
- moved R7 132.0 mm to (176.9, 92.1), turned to 90 degrees
- moved SW4 131.6 mm to (153.9, 77.0)
- moved SW3 130.1 mm to (154.1, 86.1)
- moved SW2 128.3 mm to (163.3, 117.8), turned to -90 degrees
- moved C35 122.8 mm to (140.2, 100.3), turned to 90 degrees
- moved C28 120.4 mm to (136.0, 99.1), turned to 45 degrees
- moved C27 119.7 mm to (134.7, 97.9), turned to 45 degrees
- moved D6 117.7 mm to (132.8, 122.9)
- moved P1 117.6 mm to (174.5, 109.9), turned to -90 degrees
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Connections:
- net /Power + Control/PVCC renamed /PVCC
- AE2 pad 1: Net-(AE1-OUT) -> Net-(AE2-Pad1)
- AE2 pad 2: (no net) -> GND
- C10 pad 1: GND -> GNDREF
- C10 pad 2: Net-(U2-VI) -> +BATT
- C11 pad 1: GNDREF -> GND
- C11 pad 2: +BATT -> Net-(U2-VI)
- C16 pad 1: +3.0V -> GND
- C16 pad 2: GND -> Net-(U3-VREF)
- C23 pad 1: VDDA -> +3.0V
- C24 pad 1: VDDA -> Net-(U3-CPCB)
- C24 pad 2: GND -> Net-(U3-CPCA)
- C26 pad 1: Net-(C26-Pad1) -> Net-(U3-CPOUT)
- C26 pad 2: /Audio/Lsig_in -> GND
- C27 pad 1: Net-(C27-Pad1) -> VDDA
- C27 pad 2: /Audio/Lsig_in -> GND
- C28 pad 1: Net-(C28-Pad1) -> VDDA
- C28 pad 2: /Audio/Lbass_out -> GND
- C35 pad 1: GND -> +3.0V
- C35 pad 2: Net-(U4D-IN+) -> GND
- C36 pad 1: Net-(C36-Pad1) -> Net-(U4-PA0)
- C36 pad 2: /Audio/Rbass_out -> GND
- C37 pad 1: /Audio/Lsig_out -> GND
- C37 pad 2: Net-(U5A-OUT) -> Net-(C37-Pad2)
- C38 pad 1: /Audio/Lsig_out -> Net-(AE1-OUT)
- C38 pad 2: Net-(U5A-OUT) -> Net-(AE2-Pad1)
- D5 pad 2: /Power + Control/D- -> /D-
- D6 pad 2: /Power + Control/SWDIO -> /SWDIO
- D7 pad 2: /Power + Control/D+ -> /D+
- D8 pad 2: /Power + Control/SWCLK -> /SWCLK
- D9 pad 2: /Power + Control/SWO -> /SWO
- J1 pad A6: /Power + Control/D+ -> /D+
- J1 pad A7: /Power + Control/D- -> /D-
- J1 pad B6: /Power + Control/D+ -> /D+
- J1 pad B7: /Power + Control/D- -> /D-
- R17 pad 2: /Power + Control/NRST -> /NRST
- R18 pad 2: /Power + Control/SWCLK -> /SWCLK
- R19 pad 2: /Power + Control/SWDIO -> /SWDIO
- R20 pad 2: /Power + Control/SWO -> /SWO
- R22 pad 2: Net-(U3-PH3) -> Net-(U4-PH3)
- R24 pad 1: /Audio/Lsig_in -> +3.0V
- R24 pad 2: Net-(C28-Pad1) -> Net-(U4-PA0)
- R25 pad 1: Net-(U4A-OUT) -> Net-(AE2-Pad1)
- R25 pad 2: Net-(C29-Pad1) -> GND
- SW1 pad 2: Net-(SW1-Pad2) -> Net-(C37-Pad2)
- SW2 pad 2: Net-(SW1-Pad2) -> Net-(C37-Pad2)
- SW3 pad 1: Net-(U3-PB7) -> Net-(U4-PB7)
- SW3 pad 2: Net-(U3-PB7) -> Net-(U4-PB7)
- SW4 pad 1: Net-(U3-PB8) -> Net-(U4-PB8)
- SW4 pad 2: Net-(U3-PB8) -> Net-(U4-PB8)
- TP10 pad 1: /Audio/Rbass_out -> /Rsig
- TP11 pad 1: /Audio/Rmid_out -> GND
- TP8 pad 1: /Audio/Ltreble_out -> /Lsig
- TP9 pad 1: Net-(R37-Pad2) -> GND
- U3 pad 1: +3.0V -> GND
- U3 pad 10: unconnected-(U3-PA1-Pad10) -> +3.0V
- U3 pad 11: unconnected-(U3-PA2-Pad11) -> Net-(U3-CPCA)
- U3 pad 12: /Audio/SAI_MCLK -> GND
- U3 pad 13: /Audio/Mute -> Net-(U3-CPCB)
- U3 pad 14: unconnected-(U3-PA5-Pad14) -> Net-(U3-CPOUT)
- U3 pad 15: unconnected-(U3-PA6-Pad15) -> /Rsig
- U3 pad 16: unconnected-(U3-PA7-Pad16) -> /Lsig
- U3 pad 2: unconnected-(U3-PC14-Pad2) -> VDDA
- U3 pad 3: unconnected-(U3-PC15-Pad3) -> Net-(U3-VREF)
- U3 pad 4: Net-(U3-PH3) -> /Mute
- U3 pad 5: Net-(U3-PB8) -> /SAI_FS
- U3 pad 6: Net-(D4-A) -> /SAI_SD
- U3 pad 7: /Power + Control/NRST -> /SAI_SCK
- U3 pad 8: VDDA -> /SAI_MCLK
- U3 pad 9: unconnected-(U3-PA0-Pad9) -> +3.0V
- U4 pad 1: Net-(U4A-OUT) -> +3.0V
- U4 pad 10: Net-(U4C-IN+) -> /Volume
- U4 pad 11: GND -> /Bass
- U4 pad 12: Net-(U4D-IN+) -> /SAI_MCLK
- U4 pad 13: /Audio/Ltreble_out -> /Mute
- U4 pad 14: /Audio/Ltreble_out -> /Mid
- U4 pad 2: Net-(U4A-IN-) -> unconnected-(U4-PC14-Pad2)
- U4 pad 3: Net-(U4A-IN+) -> unconnected-(U4-PC15-Pad3)
- U4 pad 4: +3.0V -> Net-(U4-PH3)
- U4 pad 5: Net-(U4B-IN+) -> Net-(U4-PB8)
- U4 pad 6: /Audio/Lmid_out -> Net-(D4-A)
- U4 pad 7: /Audio/Lmid_out -> /NRST
- U4 pad 8: Net-(U4C-OUT) -> VDDA
- U4 pad 9: Net-(U4C-IN-) -> Net-(U4-PA0)
- X1 pad 1: Net-(U3-OSC_OUT) -> Net-(U4-OSC_OUT)
- X1 pad 3: Net-(U3-OSC_IN) -> Net-(U4-OSC_IN)
Routing:
- net +3.0V: track 0.00 -> 115.5 mm, vias 0 -> 7
- net /Treble: track 0.00 -> 62.0 mm, vias 0 -> 1
- net /Mid: track 0.00 -> 60.8 mm, vias 0 -> 1
- net /D-: track 0.00 -> 59.3 mm, vias 0 -> 2
- net /D+: track 0.00 -> 56.8 mm, vias 0 -> 2
- net /Bass: track 0.00 -> 52.4 mm, vias 0 -> 1
- net /Volume: track 0.00 -> 51.0 mm, vias 0 -> 1
- net Net-(U4-PB8): track 0.00 -> 44.0 mm, vias 0 -> 2
- net Net-(U4-PB7): track 0.00 -> 39.0 mm, vias 0 -> 2
- net +5V: track 11.2 -> 41.3 mm, vias 0 -> 2
- net +BATT: track 22.8 -> 49.0 mm, vias 2 -> 3
- net VDDA: track 0.00 -> 23.3 mm, vias 0 -> 3
- net /SWDIO: track 0.00 -> 20.7 mm
- net /SWCLK: track 0.00 -> 18.9 mm, vias 0 -> 2
- net GND: track 5.53 -> 24.4 mm, vias 2 -> 58
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- added copper zone on B.Cu, net GND
- added copper zone on In1.Cu, net GND
- added copper zone on In2.Cu, net GND
- added copper zone on In2.Cu, net GNDREF
- removed copper zone on In1.Cu, net GNDREF
Other:
- board outline added: 68 x 51 mm
- board text added: "Bass"
- board text added: "Headphones Rev2 Oct 2026 Oliver Hund"
- board text added: "L+"
- board text added: "L-"
- board text added: "Mid"
- board text added: "Pause"
- board text added: "Pwr & BLE"
- board text added: "R+"
- board text added: "R-"
- board text added: "See You, Space Cactus . . ."
- board text added: "Treble"
- board text added: "Volume"
