File: headphones/headphones.kicad_sch (KiCad schematic)
At the start: 0 parts

Commit message: Final Rev2 before purchase
Parts:
- added AE1: MLPF-WB55-01E3, MLPF_WB55_01E3:MLPF-WB55-01E3_STM, symbol MLPF_WB55_01E3:MLPF-WB55-01E3
- added AE2: 2119640001, Antenna_2119640001:ANT_211964-0001_MOL, symbol Antenna_2119640001:2119640001
- added C1, C10, C12, C2, C5: 0.1uF, Capacitor_SMD:C_0603_1608Metric, symbol Device:C
- added C11, C13, C37, C7, C8: 1uF, Capacitor_SMD:C_0603_1608Metric, symbol Device:C
- added C14, C15, C6: 10uF, Capacitor_SMD:C_0603_1608Metric, symbol Device:C
- added C16: 2.2uF, Capacitor_SMD:C_0603_1608Metric, symbol Device:C_Small
- added C17: 10u, Capacitor_SMD:C_0603_1608Metric, symbol Device:C
- added C18, C19, C20, C21, C22, C23, C36: 0.1u, Capacitor_SMD:C_0603_1608Metric, symbol Device:C
- added C24: 220nF, Capacitor_SMD:C_0603_1608Metric, symbol Device:C_Small
- added C25, C26: 4.7uF, Capacitor_SMD:C_0603_1608Metric, symbol Device:C_Small
- added C27: 10n, Capacitor_SMD:C_0603_1608Metric, symbol Device:C
- added C28, C35: 1u, Capacitor_SMD:C_0603_1608Metric, symbol Device:C
- added C29, C30, C31, C32, C33, C34: 330uF, Capacitor_SMD:C_1210_3225Metric, symbol Device:C_Small
- added C3: 33nF, Capacitor_SMD:C_0603_1608Metric, symbol Device:C
- added C38: 2.7pF, Capacitor_SMD:C_0402_1005Metric, symbol Device:C_Small
- added C4: 2.2uF, Capacitor_SMD:C_0603_1608Metric, symbol Device:C
- added C9: 0.047uF, Capacitor_SMD:C_0603_1608Metric, symbol Device:C
- added D1: LED, R, Resistor_SMD:R_1206_3216Metric, symbol Device:LED
- added D2, D3: (no value), Diode_SMD:D_SOD-323F, symbol Device:D_Schottky
- added D4: LED, O, Resistor_SMD:R_1206_3216Metric, symbol Device:LED
- added D5, D6, D7, D8, D9: SD03CQ_SOD323, Diode_SMD:D_SOD-323, symbol Diode:SD05_SOD323
- added FB1: 120R, Resistor_SMD:R_0603_1608Metric, symbol Device:FerriteBead
- added J1: UJ20-C-H-G-SMT-1-P16-TR, USBC_Connector:SAMESKY_UJ20-C-H-G-SMT-1-P16-TR, symbol UJ20-C-H-G-SMT-1-P16-TR:UJ20-C-H-G-SMT-1-P16-TR
- added J2: Conn_ARM_SWD_TagConnect_TC2030-NL, Connector:Tag-Connect_TC2030-IDC-NL_2x03_P1.27mm_Vertical, symbol Connector:Conn_ARM_SWD_TagConnect_TC2030-NL
- added L1: 10uH, Inductor_SMD:L_0805_2012Metric, symbol Device:L
- added P1: S2B-PH-SM4-TB, S2B_PH_SM4_TB:S2B-PH-SM4-TB, symbol S2B_PH_SM4_TB:S2B-PH-SM4-TB
- added R1: 47k, Resistor_SMD:R_0603_1608Metric, symbol Device:R
- added R10: 5, Resistor_SMD:R_0603_1608Metric, symbol Device:R
- added R11, R12, R17, R18, R19, R20: 150, Resistor_SMD:R_0603_1608Metric, symbol Device:R
- added R13: 13k, Resistor_SMD:R_0603_1608Metric, symbol Device:R
- added R14: 1k, Resistor_SMD:R_0603_1608Metric, symbol Device:R
- added R15: 8.2k, Resistor_SMD:R_0603_1608Metric, symbol Device:R
- added R16: 56k, Resistor_SMD:R_0603_1608Metric, symbol Device:R
- added R2: 15k, Resistor_SMD:R_0603_1608Metric, symbol Device:R
- added R21: 47m, Resistor_SMD:R_0805_2012Metric, symbol Device:R
- added R22: 10k, Resistor_SMD:R_0603_1608Metric, symbol Device:R
- added R23: 330, Resistor_SMD:R_0603_1608Metric, symbol Device:R
- added R24: P120PK-Y25BR10K, Pot1gang10k_P120PK_Y25BR10K:POT_P120PK-x25_TTE, symbol Pot1gang10k_P120PK_Y25BR10K:P120PK-Y25BR10K
- added R25: 0, Resistor_SMD:R_0402_1005Metric, symbol Device:R
- added R3, R6, R7: 5.1k, Resistor_SMD:R_0603_1608Metric, symbol Device:R
- added R4: 30k, Resistor_SMD:R_0603_1608Metric, symbol Device:R
- added R5: 20m, Resistor_SMD:R_0603_1608Metric, symbol Device:R
- added R8: 2, Resistor_SMD:R_0603_1608Metric, symbol Device:R
- added R9: 750, Resistor_SMD:R_0805_2012Metric, symbol Device:R
- added S1: SLW-1478144-5A-S-D, SP4T_SLW_1478144_5A_S_D:SW_SLW-1478144-5A-S-D, symbol SP4T_SLW_1478144_5A_S_D:SLW-1478144-5A-S-D
- added SW1, SW2: OS102011MS2QN1, SPDT_OS102011MS2QN1:SPDT_OS102011_CNK, symbol SPDT_OS102011MS2QN1.zip:OS102011MS2QN1
- added SW3, SW4: SW_MEC_5E, OFF-Mom_PTS526_SM15_SMTR2_LFS:SON4_PTS526 SM15 SMTR2 LFS_CNK, symbol Switch:SW_MEC_5E
- added TH1: 10k, Resistor_SMD:R_0603_1608Metric, symbol Device:Thermistor
- added TP1, TP2, TP3, TP4, TP5, TP6, TP7: TestPoint, TestPoint:TestPoint_Pad_D1.5mm, symbol Connector:TestPoint
- added TP10: +RDriver, TestPoint:TestPoint_Pad_D1.5mm, symbol Connector:TestPoint
- added TP11: -RDriver, TestPoint:TestPoint_Pad_D1.5mm, symbol Connector:TestPoint
- added TP8: +LDriver, TestPoint:TestPoint_Pad_D1.5mm, symbol Connector:TestPoint
- added TP9: -LDriver, TestPoint:TestPoint_Pad_D1.5mm, symbol Connector:TestPoint
- added U1: BQ24133RGY, Package_DFN_QFN:Texas_RGY_R-PVQFN-N24_EP2.05x3.1mm, symbol Battery_Management:BQ24133RGY
- added U2: AP2127N-3.0, Package_TO_SOT_SMD:SOT-23, symbol Regulator_Linear:AP2127N-3.0
- added U3: NAU8402WG, DAC_NAU8402WG:TSSOP16_NAU8402_NUV, symbol DAC_NAU8402WG:NAU8402WG
- added U4: STM32WB55CCUx, Package_DFN_QFN:QFN-48-1EP_7x7mm_P0.5mm_EP5.6x5.6mm, symbol MCU_ST_STM32WB:STM32WB55CCUx
- added X1: NX2016SA-32MHZ-EXS00A-CS06654, NX2016SA_32MHZ_EXS00A_CS06654:NX2016SA_NDK, symbol NX2016SA_32MHZ_EXS00A_CS06654:NX2016SA-32MHZ-EXS00A-CS06654
Connections:
- net +3.0V: now also C13.2, C17.1, C18.1, C19.1, C20.1, C21.1, C22.1, C23.1, C25.1, C35.1, FB1.2, R11.2, R24.1, TP4.1, U2.2 (VO), U3.10 (LINEVDD), U3.9 (VDDB), U4.1 (VBAT), U4.20 (VDD), U4.23 (VDDRF), U4.31 (VFBSMPS), U4.33 (VLXSMPS), U4.34 (VDDSMPS), U4.35 (VDD), U4.48 (VDD)
- net GND: now also AE1.A2 (GND4), AE1.B1 (GND3), AE1.B2 (GND2), AE1.B3 (GND1), C1.2, C11.1, C13.1, C14.1, C15.1, C16.1, C17.2, C18.2, C19.2, C20.2, C21.2, C22.2, C23.2, C25.2, C26.2, C27.2, C28.2, C35.2, C36.2, C37.1, C4.2, C5.2, C6.2, C7.1, D5.1 (A1), D6.1 (A1), D7.1 (A1), D8.1 (A1), D9.1 (A1), J1.A1_B12 (GND), J1.B1_A12 (GND__1), J1.SH1 (SHIELD), J1.SH2 (SHIELD__1), J1.SH3 (SHIELD__2), J1.SH4 (SHIELD__3), P1.2, R12.1, R22.1, R23.2, R24.3, R25.2, R6.2, R7.2, S1.3, SW3.3 (K), SW3.4 (A), SW4.3 (K), SW4.4 (A), TP11.1, TP9.1, U1.22 (PGND), U1.23 (PGND), U2.1 (GND), U3.1 (VSSA), U3.12 (LINEGND), U4.22 (VSSRF), U4.32 (VSSSMPS), U4.40 (VDDUSB), U4.49 (VSS), X1.2, X1.4
- net VDDA: now also C27.1, C28.1, FB1.1, TP7.1, U3.2 (VDDA), U4.8 (VDDA)
- new net: C11.2, SW2.3, U2.3 (VI)
- new net: C7.2, U1.20 (REGN)
- new net: C29.1, C30.1, C31.1, TP8.1
- new net: C12.1, L1.2, R21.1, U1.16 (SRP)
- new net: D1.1 (K), U1.9 (STAT)
- new net: D1.2 (A), R9.1
- new net: C36.1, R24.2, U4.9 (PA0)
- new net: C9.1, L1.1, U1.1 (SW), U1.24 (SW)
- new net: R3.2, R4.1, TH1.1, U1.10 (TS)
- new net: C3.1, U1.11 (TTC)
- new net: R13.2, R14.1, U1.13 (ISET)
- new net: R15.2, R16.1, U1.17 (ACSET)
- new net: R1.2, R2.1, U1.18 (OVPSET)
- new net: C9.2, U1.21 (BTST)
- new net: C5.1, D3.1 (K), R10.2, TP3.1, U1.4 (AVCC)
- new net: C24.2, U3.11 (CPCA)
- new net: C24.1, U3.13 (CPCB)
- new net: C26.1, U3.14 (CPOUT)
- new net: C16.2, U3.3 (VREF)
- new net: D4.1 (K), R23.1
- new net: J2.4 (SWCLK), R18.1
- new net: J1.B5 (CC2), R7.1
- new net: C32.1, C33.1, C34.1, TP10.1
- new net: J1.A5 (CC1), R6.1
- new net: C4.1, R8.2
- new net: AE1.A3 (IN), U4.21 (RF1)
- new net: U4.24 (OSC_OUT), X1.1
- new net: U4.25 (OSC_IN), X1.3
- new net: R22.2, U4.4 (PH3)
- new net: SW3.1, SW3.2, U4.47 (PB7)
- new net: SW4.1, SW4.2, U4.5 (PB8)
- new net: D4.2 (A), U4.6 (PB9)
- new net: D2.1 (K), R10.1
- new net: C37.2, SW1.2, SW2.2
- new net: J2.1 (VCC), R11.1
- new net: J2.3 (~{RESET}), R17.1
- new net: AE1.A1 (OUT), C38.1
- new net: J2.6 (SWO), R20.1
- new net: AE2.1, C38.2, R25.1
- new net: J2.2 (SWDIO), R19.1
- new net: J2.5 (GND), R12.2
- new net +3.3V, ref: C8.2, R13.1, R15.1, R3.1, R9.2, U1.12 (VREF)
- new net +5V: C2.1, D2.2 (A), J1.A4_B9 (VBUS), J1.B4_A9 (VBUS__1), R1.1, R5.1, R8.1, SW1.3, TP1.1, U1.6 (ACP)
- new net +BATT: C10.2, C12.2, C14.2, C15.2, D3.2 (A), P1.1, R21.2, SW1.1, TP2.1, U1.15 (SRN)
- new net Bass: S1.2, U4.11 (PA2)
- new net D+: D7.2 (A2), J1.A6 (DP1), J1.B6 (DP2), U4.38 (PA12)
- new net D-: D5.2 (A2), J1.A7 (DN1), J1.B7 (DN2), U4.37 (PA11)
- new net GNDREF: C10.1, C3.2, C8.1, R14.2, R16.2, R2.2, R4.2, TH1.2, U1.14 (CELL), U1.25 (AGND)
- new net Lsig: C29.2, C30.2, C31.2, TP5.1, U3.16 (LLINEOU)
- new net Mid: S1.5, U4.14 (PA5)
- new net Mute: U3.4 (MUTEB), U4.13 (PA4)
- new net NRST: R17.2, U4.7 (NRST)
- new net PVCC: C1.1, C2.2, C6.1, R5.2, U1.2 (PVCC), U1.3 (PVCC), U1.5 (ACN)
- new net Rsig: C32.2, C33.2, C34.2, TP6.1, U3.15 (RLINEOUT)
- new net SAI_FS: U3.5 (FS), U4.18 (PA9)
- new net SAI_MCLK: U3.8 (MCLK), U4.12 (PA3)
- new net SAI_SCK: U3.7 (BCLK), U4.17 (PA8)
- new net SAI_SD: U3.6 (DACIN), U4.36 (PA10)
- new net SWCLK: D8.2 (A2), R18.2, U4.41 (PA14)
- new net SWDIO: D6.2 (A2), R19.2, U4.39 (PA13)
- new net SWO: D9.2 (A2), R20.2, U4.43 (PB3)
- new net Treble: S1.6, U4.15 (PA6)
- new net Volume: S1.1, U4.10 (PA1)
- no-connect marks 0 -> 17
Other:
- removed sheet Audio
- removed sheet Power + Control
- note added: "BLE Pair"
- note added: "Charging Interface"
- note added: "Control for S1 parameters"
- note added: "DAC & Drivers"
- note added: "Drivers"
- note added: "Headphone Rev2; Oliver Hund"
- note added: "LPF and matching network RF1 - AE1 60Ohm trace AE1 - AE2 20Ohm trace"
- note added: "Pause"
- note added: "Power & LDO"
- note added: "STM32WB55c"
- note added: "SW2: 1&2 battery is power source (+3.0V) SW2: 2&3 USBC is power source (+5V) SW1: 1&2 HighZ, no power to MCU SW1: 2&3 MCU power from SW2"
- note added: "SWD"
- note added: "Switch for: Volume Bass Mids Treble"
- note added: "Test LED"
- note added: "USBC"
- note removed: "Headphone Rev1; Oliver Hund"
